File: hardware/pcb-carrier/kbdrelay-carrier/kbdrelay-carrier-test2.kicad_pcb (KiCad board)
At the start: 2 copper layers, 88 x 55 mm, 22 parts, among them J1 UART_KBD, J2 UART_TGT, J3 5V_IN, U1 ESP32-S3-Zero, U2 ESP32-S3-Zero

Commit message: chore(pcb): clear fab/, derive LCD crop from the board, document refill trap
fab/ is emptied: it held two naming conventions from two different exports
(GUI .gbr and CLI protel-style), which is the stale-artwork trap in a new
outfit. Everything there is regenerable; user is regenerating from test2.

make_lcd_art.sh now takes a board path and derives the crop window from the
real Edge.Cuts bounding box instead of hardcoded pixel offsets, so it follows
the board instead of silently mis-registering if the outline moves.

BUILD.md gains two warnings earned the hard way:
- refill the GND zone before every export; KiCad does not do it automatically
  and only DRC notices. A stale fill had the pour 0.15 mm from live copper
  while the rule said 1.4 mm.
- test2 is the board of record; the script-generated board does not match it.
Parts:
- moved F1 2.00 mm to (110.5, 117.5)
- moved C1 1.68 mm to (114.2, 127.2)
Routing:
- net /+5V_PROT: track 23.0 -> 29.2 mm
- net Net-(U1-GPIO5): track 26.9 -> 29.2 mm
- net GND: track 9.58 -> 11.8 mm
- net Net-(U2-GPIO4): track 20.8 -> 22.5 mm
- net /DRDY_TGT: track 42.8 -> 44.4 mm
- net /+5V_KBD: track 6.86 -> 5.53 mm
- net Net-(U2-GPIO5): track 15.9 -> 17.2 mm
- net /CS_TGT: track 28.9 -> 30.1 mm
- net Net-(U2-RX): track 26.4 -> 27.2 mm
- net Net-(J2-Pin_2): track 4.89 -> 5.55 mm
Changed lines of the file:
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@@
 			(outputformat 1)
 			(mirror no)
-			(drillshape 1)
+			(drillshape 0)
 			(scaleselection 1)
 			(outputdirectory "../fab/gerbers/")
@@
 	(footprint "kbdrelay:PPTC_Littelfuse_60R_P5.08mm"
 		(layer "F.Cu")
-		(at 110.5 119.5 180)
+		(at 110.5 117.5 180)
 		(descr "Littelfuse 60R series radial-leaded PPTC. Silkscreen sized for 60R090 (Ihold 0.90 A / Itrip 1.80 A, 60 V, body 11.2 x 3.1 mm max); also fits smaller bodies in the family (60R050 is 7.9 mm) since all share 0.20 in / 5.08 mm lead centres and 0.51 mm lead dia. Pads/drills enlarged to 2.0 mm / 1.0 mm for single-sided home etching (0.5 mm annular ring, same drill bit as the module pads). Datasheet: https://www.littelfuse.com/products/fuses-overcurrent-protection/polyswitch-resettable-pptc-devices/radial-leaded-polyswitch-resettable-pptc-devices/60r")
 		(tags "pptc resettable fuse polyfuse littelfuse 60r radial tht")
@@
 	(footprint "Capacitor_THT:CP_Radial_D10.0mm_P5.00mm"
 		(layer "F.Cu")
-		(at 112.75 126.5)
+		(at 114.25 127.25)
 		(descr "CP, Radial series, Radial, pin pitch=5.00mm, diameter=10mm, height=16mm, Electrolytic Capacitor")
 		(tags "CP Radial series Radial pin pitch 5.00mm diameter 10mm height 16mm Electrolytic Capacitor")
@@
 		)
 		(property "Value" "ESP32-S3-Zero"
-			(at 9.09 24.94 180)
+			(at 10.03 27.25 270)
 			(unlocked yes)
 			(layer "F.Fab")
@@
 		)
 		(fp_text user "${REFERENCE}"
-			(at 9.09 26.44 180)
+			(at 10.408871 25.204516 270)
 			(unlocked yes)
 			(layer "F.Fab")
@@
 		(start 120.5 119.5)
 		(end 124.45 124.25)
-		(width 1.5)
+		(width 1)
 		(layer "B.Cu")
 		(net "/+5V_PROT")
 	)
 	(segment
-		(start 112.75 126.5)
-		(end 113.04 126.21)
-		(width 1.5)
+		(start 110.25 120.5)
+		(end 114.25 124.5)
+		(width 1)
 		(layer "B.Cu")
 		(net "/+5V_PROT")
 	)
 	(segment
-		(start 113.04 119.5)
-		(end 120.5 119.5)
-		(width 1.5)
+		(start 124.45 124.25)
+		(end 124.5 126.5)
+		(width 1)
 		(layer "B.Cu")
 		(net "/+5V_PROT")
 	)
 	(segment
-		(start 113.04 126.21)
-		(end 113.04 119.5)
-		(width 1.5)
+		(start 113.04 117.5)
+		(end 115.04 119.5)
+		(width 1)
 		(layer "B.Cu")
 		(net "/+5V_PROT")
 	)
 	(segment
-		(start 124.45 124.25)
-		(end 124.5 126.5)
-		(width 1.5)
+		(start 113.04 117.5)
+		(end 110.25 120.5)
+		(width 1)
+		(layer "B.Cu")
+		(net "/+5V_PROT")
+	)
+	(segment
+		(start 115.04 119.5)
+		(end 120.5 119.5)
+		(width 1)
 		(layer "B.Cu")
 		(net "/+5V_PROT")
 	)
 	(segment
+		(start 114.25 124.5)
+		(end 114.25 127.25)
+		(width 1)
+		(layer "B.Cu")
+		(net "/+5V_PROT")
+	)
+	(segment
+		(start 107.59 117.13)
+		(end 107.96 117.5)
+		(width 1)
+		(layer "B.Cu")
+		(net "/+5V_KBD")
+	)
+	(segment
 		(start 107.59 112.65)
-		(end 107.96 119.5)
-		(width 1.5)
+		(end 107.59 117.13)
+		(width 1)
+		(layer "B.Cu")
+		(net "/+5V_KBD")
+	)
+	(segment
+		(start 107.96 113.02)
+		(end 107.59 112.65)
+		(width 0.8)
 		(layer "B.Cu")
 		(net "/+5V_KBD")
@@
 		(start 164.5 119.5)
 		(end 168.5 119.5)
-		(width 0.8)
+		(width 1)
 		(layer "B.Cu")
 		(net "Net-(J2-Pin_1)")
 	)
 	(segment
-		(start 166.05 122.25)
-		(end 168.5 124.5)
-		(width 0.8)
+		(start 164.5 122.04)
+		(end 167.25 122)
+		(width 1)
 		(layer "B.Cu")
 		(net "Net-(J2-Pin_2)")
 	)
 	(segment
-		(start 164.5 122.04)
-		(end 166.05 122.25)
-		(width 0.8)
+		(start 167.25 122)
+		(end 168.5 124.5)
+		(width 1)
 		(layer "B.Cu")
 		(net "Net-(J2-Pin_2)")
 	)
 	(segment
+		(start 137.5 122.04)
+		(end 139.21 122.04)
+		(width 1)
+		(layer "B.Cu")
+		(net "GND")
+	)
+	(segment
 		(start 110.13 112.65)
 		(end 110.13 109.63)
@@
 	)
 	(segment
-		(start 186.87 97.35)
-		(end 186.87 95.12)
-		(width 0.65)
+		(start 129.5 126.5)
+		(end 131 126.5)
+		(width 1)
 		(layer "B.Cu")
 		(net "GND")
 	)
 	(segment
-		(start 117.75 126.5)
-		(end 120.5 126.5)
+		(start 119.25 127.25)
+		(end 121 127.25)
 		(width 1)
 		(layer "B.Cu")
@@
 	)
 	(segment
-		(start 191.41 111.66)
-		(end 191.41 113.418428)
+		(start 186.87 97.35)
+		(end 186.87 95.12)
 		(width 1)
 		(layer "B.Cu")
-		(net "Net-(U2-RX)")
+		(net "GND")
 	)
 	(segment
-		(start 191.41 113.418428)
+		(start 191.5 115.25)
 		(end 180.328428 124.5)
 		(width 1)
@@
 	)
 	(segment
-		(start 180.328428 124.5)
-		(end 178.66 124.5)
+		(start 189.5 109.75)
+		(end 191.5 111.5)
 		(width 1)
 		(layer "B.Cu")
@@
 	)
 	(segment
-		(start 189.5 109.75)
-		(end 191.41 111.66)
+		(start 180.328428 124.5)
+		(end 178.66 124.5)
+		(width 1)
+		(layer "B.Cu")
+		(net "Net-(U2-RX)")
+	)
+	(segment
+		(start 191.5 111.5)
+		(end 191.5 115.25)
 		(width 1)
 		(layer "B.Cu")
@@
 	)
 	(segment
-		(start 159.66 96.5)
-		(end 157.65 98.65)
+		(start 168.05 113.45)
+		(end 169.09 112.59)
 		(width 1)
 		(layer "B.Cu")
@@
 	)
 	(segment
-		(start 157.65 98.65)
-		(end 157.65 112.45)
+		(start 159.66 96.5)
+		(end 157 98.75)
 		(width 1)
 		(layer "B.Cu")
@@
 	)
 	(segment
-		(start 168.05 113.45)
-		(end 169.09 112.59)
+		(start 157 98.75)
+		(end 157 112.5)
 		(width 1)
 		(layer "B.Cu")
@@
 	)
 	(segment
-		(start 158.65 113.45)
-		(end 168.05 113.45)
+		(start 157 112.5)
+		(end 157.75 113.45)
 		(width 1)
 		(layer "B.Cu")
@@
 	)
 	(segment
-		(start 157.65 112.45)
-		(end 158.65 113.45)
+		(start 157.75 113.45)
+		(end 168.05 113.45)
 		(width 1)
 		(layer "B.Cu")
@@
 	)
 	(segment
-		(start 160.79137 111.5)
-		(end 174.17 98.12137)
+		(start 174.17 97.35)
+		(end 174.17 100.92)
 		(width 1)
 		(layer "B.Cu")
@@
 	)
 	(segment
-		(start 174.17 98.12137)
-		(end 174.17 97.35)
+		(start 174.17 100.92)
+		(end 163.75 111.5)
 		(width 1)
 		(layer "B.Cu")
@@
 	)
 	(segment
-		(start 159.66 111.5)
-		(end 160.79137 111.5)
+		(start 163.75 111.5)
+		(end 159.66 111.5)
 		(width 1)
 		(layer "B.Cu")
@@
 	)
 	(segment
-		(start 155.75 113.5)
-		(end 157.75 115.75)
+		(start 154.75 113.5)
+		(end 157.25 116.25)
 		(width 1)
 		(layer "B.Cu")
@@
 	)
 	(segment
-		(start 170.5 115.75)
-		(end 171.63 112.59)
+		(start 159.66 91.5)
+		(end 154.5 95.75)
 		(width 1)
 		(layer "B.Cu")
@@
 	)
 	(segment
-		(start 157.75 115.75)
-		(end 170.5 115.75)
+		(start 169 116.25)
+		(end 171.63 112.59)
 		(width 1)
 		(layer "B.Cu")
@@
 	)
 	(segment
-		(start 159.66 91.5)
-		(end 155.5 95.75)
+		(start 157.25 116.25)
+		(end 169 116.25)
 		(width 1)
 		(layer "B.Cu")
@@
 	)
 	(segment
-		(start 155.5 95.75)
-		(end 155.75 113.5)
+		(start 154.5 95.75)
+		(end 154.75 113.5)
 		(width 1)
 		(layer "B.Cu")
@@
 	)
 	(segment
-		(start 130.85 106.65)
+		(start 131.25 104.5)
+		(end 147.5 104.5)
+		(width 1)
+		(layer "B.Cu")
+		(net "Net-(U1-GPIO5)")
+	)
+	(segment
+		(start 147.5 104.5)
 		(end 149.5 106.5)
 		(width 1)
@@
 	(segment
 		(start 125.65 111.85)
-		(end 130.85 106.65)
+		(end 131.25 104.5)
 		(width 1)
 		(layer "B.Cu")
@@
 	(segment
 		(start 171.63 97.35)
-		(end 171.63 97.638428)
+		(end 171.63 99.88)
 		(width 1)
 		(layer "B.Cu")
@@
 	)
 	(segment
-		(start 171.63 97.638428)
-		(end 169.768428 99.5)
+		(start 165.01 106.5)
+		(end 171.63 99.88)
 		(width 1)
 		(layer "B.Cu")
@@
 	)
 	(segment
-		(start 168 99.5)
-		(end 161 106.5)
+		(start 159.66 106.5)
+		(end 165.01 106.5)
 		(width 1)
 		(layer "B.Cu")
@@
 	)
 	(segment
-		(start 169.768428 99.5)
-		(end 168 99.5)
+		(start 150 109)
+		(end 152 107.25)
 		(width 1)
 		(layer "B.Cu")
-		(net "Net-(U2-GPIO5)")
+		(net "Net-(U1-GPIO6)")
 	)
 	(segment
-		(start 161 106.5)
-		(end 159.66 106.5)
+		(start 132.5 109)
+		(end 150 109)
 		(width 1)
 		(layer "B.Cu")
-		(net "Net-(U2-GPIO5)")
+		(net "Net-(U1-GPIO6)")
 	)
 	(segment
@@
 	)
 	(segment
-		(start 150.75 108.5)
-		(end 152 107.25)
-		(width 1)
-		(layer "B.Cu")
-		(net "Net-(U1-GPIO6)")
-	)
-	(segment
 		(start 127.91 112.65)
-		(end 132.65 108.45)
+		(end 132.5 109)
 		(width 1)
 		(layer "B.Cu")
@@
 	)
 	(segment
-		(start 132.65 108.45)
-		(end 150.75 108.5)
-		(width 1)
-		(layer "B.Cu")
-		(net "Net-(U1-GPIO6)")
-	)
-	(segment
 		(start 165.15 97.35)
 		(end 169.09 97.35)
@@
 		(start 183.85 114.65)
 		(end 188.05 114.65)
-		(width 0.8)
+		(width 1)
 		(layer "B.Cu")
 		(net "Net-(U2-TX)")
@@
 		(start 188.05 114.65)
 		(end 189.41 112.59)
-		(width 0.8)
+		(width 1)
 		(layer "B.Cu")
 		(net "Net-(U2-TX)")
@@
 		(start 178.66 119.5)
 		(end 183.85 114.65)
-		(width 0.8)
+		(width 1)
 		(layer "B.Cu")
 		(net "Net-(U2-TX)")
@@
 		)
 		(min_thickness 0.4)
-		(fill yes
+		(fill
 			(thermal_gap 0.4)
 			(thermal_bridge_width 0.8)

Commit message: Working 0.1 board
Parts:
- moved D1 1.00 mm to (120.5, 118.5)
- moved C1 0.75 mm to (114.2, 126.5)
Routing:
- net GND: track 11.8 -> 0.00 mm
- net /+5V_PROT: track 29.2 -> 26.6 mm
Changed lines of the file:
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@@
 		(capping no)
 		(filling no)
-		(zone_defaults)
 		(pcbplotparams
 			(layerselection 0x00000000_00000000_55555555_5755f5ff)
@@
 	(footprint "Capacitor_THT:CP_Radial_D10.0mm_P5.00mm"
 		(layer "F.Cu")
-		(at 114.25 127.25)
+		(at 114.25 126.5)
 		(descr "CP, Radial series, Radial, pin pitch=5.00mm, diameter=10mm, height=16mm, Electrolytic Capacitor")
 		(tags "CP Radial series Radial pin pitch 5.00mm diameter 10mm height 16mm Electrolytic Capacitor")
@@
 	(footprint "Diode_THT:D_DO-201AD_P12.70mm_Horizontal"
 		(layer "F.Cu")
-		(at 120.5 119.5)
+		(at 120.5 118.5)
 		(descr "Diode, DO-201AD series, Axial, Horizontal, pin pitch=12.7mm, length*diameter=9.5*5.2mm^2, http://www.diodes.com/_files/packages/DO-201AD.pdf")
 		(tags "Diode DO-201AD series Axial Horizontal pin pitch 12.7mm  length 9.5mm diameter 5.2mm")
@@
 	)
 	(segment
-		(start 120.5 119.5)
-		(end 124.45 124.25)
-		(width 1)
-		(layer "B.Cu")
-		(net "/+5V_PROT")
-	)
-	(segment
-		(start 110.25 120.5)
-		(end 114.25 124.5)
+		(start 114.25 126.5)
+		(end 114.25 118.71)
 		(width 1)
 		(layer "B.Cu")
@@
 	)
 	(segment
-		(start 113.04 117.5)
-		(end 115.04 119.5)
+		(start 114.25 118.71)
+		(end 113.04 117.5)
 		(width 1)
 		(layer "B.Cu")
@@
 	)
 	(segment
-		(start 113.04 117.5)
-		(end 110.25 120.5)
+		(start 119.5 117.5)
+		(end 120.5 118.5)
 		(width 1)
 		(layer "B.Cu")
@@
 	)
 	(segment
-		(start 115.04 119.5)
-		(end 120.5 119.5)
+		(start 120.5 118.5)
+		(end 124.45 124.25)
 		(width 1)
 		(layer "B.Cu")
@@
 	)
 	(segment
-		(start 114.25 124.5)
-		(end 114.25 127.25)
+		(start 113.04 117.5)
+		(end 119.5 117.5)
 		(width 1)
 		(layer "B.Cu")
@@
 	)
 	(segment
-		(start 137.5 122.04)
-		(end 139.21 122.04)
-		(width 1)
-		(layer "B.Cu")
-		(net "GND")
-	)
-	(segment
-		(start 110.13 112.65)
-		(end 110.13 109.63)
-		(width 1)
-		(layer "B.Cu")
-		(net "GND")
-	)
-	(segment
-		(start 164.5 124.58)
-		(end 162.92 124.58)
-		(width 1)
-		(layer "B.Cu")
-		(net "GND")
-	)
-	(segment
-		(start 129.5 126.5)
-		(end 131 126.5)
-		(width 1)
-		(layer "B.Cu")
-		(net "GND")
-	)
-	(segment
-		(start 119.25 127.25)
-		(end 121 127.25)
-		(width 1)
-		(layer "B.Cu")
-		(net "GND")
-	)
-	(segment
-		(start 186.87 97.35)
-		(end 186.87 95.12)
-		(width 1)
-		(layer "B.Cu")
-		(net "GND")
-	)
-	(segment
 		(start 191.5 115.25)
 		(end 180.328428 124.5)
@@
 	)
 	(segment
-		(start 133.199999 119.5)
+		(start 133.2 118.5)
 		(end 137.5 119.5)
 		(width 1.5)
@@
 	)
 	(segment
-		(start 131.25 104.5)
-		(end 147.5 104.5)
+		(start 126 109.25)
+		(end 131.25 104.5)
 		(width 1)
 		(layer "B.Cu")
@@
 	)
 	(segment
-		(start 125.65 111.85)
-		(end 131.25 104.5)
+		(start 125.37 112.65)
+		(end 126 109.25)
 		(width 1)
 		(layer "B.Cu")
@@
 	)
 	(segment
-		(start 125.37 112.65)
-		(end 125.65 111.85)
+		(start 131.25 104.5)
+		(end 147.5 104.5)
 		(width 1)
 		(layer "B.Cu")
@@
 		)
 		(min_thickness 0.4)
-		(fill
+		(fill yes
 			(thermal_gap 0.4)
 			(thermal_bridge_width 0.8)
